Commit message: Robot sessions 29 Oct: AppWalk/SwayStep, fall recovery, mirror, sim-to-real logging
Hardware milestones A-C on the real robot (192.168.89.74, firmware 2.8.0.55):
- IMU emulation remapped to the measured chip axes (accel and gyro x right, y up,
  z back); .hts frame index 1-based like the robot's files.
- Fall recovery (yanshee_sim/recovery.py): posture from euler-x/y, fall vs laid
  down, Base_GetupF + lock check + reset face down, GetupRear on the back; GUI
  Auto get-up. Firmware fall management concluded OFF. Mat get-up parked
  (docs/GETUP_ON_MATS.md, tools/getup_lab.py, tools/getup_research/).
- Walking: AppWalk replicates the mobile app's protocol (captured); SwayStep is
  our gait. GUI "Robot walk" selects either; SwayStep streams to /hal_angles_set
  50/s through the robot link (yanshee_sim/robot_stream.py: a python2 ROS node
  started over ssh; hal ignores NeckLR on that topic). Fall statistics per
  method (walkstats.py, tools/walk_stats.py), tools/joystick.py,
  tools/record_gait.py, tools/walk_trial.py.
- With a robot connected the sim mirrors it kinematically (encoders + IMU,
  physics paused, SimRobot.set_mirror); Both mode no longer runs SwayStep beside
  AppWalk. A hidden shadow simulator (shadow.py) gets the robot's servo frames.
- Sim-to-real logs: the robot logs on board with its own clock (IMU, encoders
  via hal_servo_read, every frame, hal read-service monitor, /rosout_agg); the
  laptop logs the shadow, mirror input and clock pings; fetched on disconnect
  (tools/fetch_robot_logs.py), merged by tools/sim2real_report.py.
- tools/robot_checks.py: latency, imu, gyro, fall, servo, gait, inspect modes.

From a parallel session: physical link inertias (no lumped rotor term), servo
torque 1.15 N*m fitted to the robot's get-ups, model/scene_mat.xml (grippy mat),
tools/getup_compare.py.

Tests: 157; test_gait_direction_changes_do_not_tip still fails intermittently in
full runs (passes alone).

Co-Authored-By: Claude Opus 5.5 <noreply@anthropic.com>

File: ros2_ws/src/yanshee_description/urdf/yanshee.urdf (robot description, URDF)
Before this commit: robot yanshee, 20 links, 19 joints
Joints:
- joint LeftAnkleFB: limit lower=0 upper=3.14159 effort=2.0 velocity=6.0 -> lower=0 upper=3.14159 effort=1.15 velocity=6.0
- joint LeftAnkleUD: limit lower=0 upper=2.00713 effort=2.0 velocity=6.0 -> lower=0 upper=2.00713 effort=1.15 velocity=6.0
- joint LeftElbowFlex: limit lower=0 upper=3.14159 effort=2.0 velocity=6.0 -> lower=0 upper=3.14159 effort=1.15 velocity=6.0
- joint LeftHipFB: limit lower=0 upper=2.96706 effort=2.0 velocity=6.0 -> lower=0 upper=2.96706 effort=1.15 velocity=6.0
- joint LeftHipLR: limit lower=1.0472 upper=3.14159 effort=2.0 velocity=6.0 -> lower=1.0472 upper=3.14159 effort=1.15 velocity=6.0
- joint LeftKneeFlex: limit lower=0 upper=3.14159 effort=2.0 velocity=6.0 -> lower=0 upper=3.14159 effort=1.15 velocity=6.0
- joint LeftShoulderFlex: limit lower=0 upper=3.14159 effort=2.0 velocity=6.0 -> lower=0 upper=3.14159 effort=1.15 velocity=6.0
- joint LeftShoulderRoll: limit lower=0 upper=3.14159 effort=2.0 velocity=6.0 -> lower=0 upper=3.14159 effort=1.15 velocity=6.0
- joint NeckLR: limit lower=0.261799 upper=2.87979 effort=2.0 velocity=6.0 -> lower=0.261799 upper=2.87979 effort=1.15 velocity=6.0
- joint RightAnkleFB: limit lower=0 upper=3.14159 effort=2.0 velocity=6.0 -> lower=0 upper=3.14159 effort=1.15 velocity=6.0
- joint RightAnkleUD: limit lower=1.13446 upper=3.14159 effort=2.0 velocity=6.0 -> lower=1.13446 upper=3.14159 effort=1.15 velocity=6.0
- joint RightElbowFlex: limit lower=0 upper=3.14159 effort=2.0 velocity=6.0 -> lower=0 upper=3.14159 effort=1.15 velocity=6.0
- joint RightHipFB: limit lower=0.174533 upper=3.14159 effort=2.0 velocity=6.0 -> lower=0.174533 upper=3.14159 effort=1.15 velocity=6.0
- joint RightHipLR: limit lower=0 upper=2.0944 effort=2.0 velocity=6.0 -> lower=0 upper=2.0944 effort=1.15 velocity=6.0
- joint RightKneeFlex: limit lower=0 upper=3.14159 effort=2.0 velocity=6.0 -> lower=0 upper=3.14159 effort=1.15 velocity=6.0
- joint RightShoulderFlex: limit lower=0 upper=3.14159 effort=2.0 velocity=6.0 -> lower=0 upper=3.14159 effort=1.15 velocity=6.0
- joint RightShoulderRoll: limit lower=0 upper=3.14159 effort=2.0 velocity=6.0 -> lower=0 upper=3.14159 effort=1.15 velocity=6.0
